Commit message: Fix urdf loading

File: resource/ec63.urdf (robot description, URDF)
Before this commit: robot ec63, 0 links, 0 joints
Links:
- added link base_link, mass 0.3647; collision mesh filename=package://elite_description/meshes/ec63/base_link.STL; visual mesh filename=package://elite_description/meshes/ec63/base_link.STL
- added link flan
- added link link1, mass 1.0468989469595; collision mesh filename=package://elite_description/meshes/ec63/link1.STL; visual mesh filename=package://elite_description/meshes/ec63/link1.STL
- added link link2, mass 2.6439; collision mesh filename=package://elite_description/meshes/ec63/link2.STL; visual mesh filename=package://elite_description/meshes/ec63/link2.STL
- added link link3, mass 1.4492; collision mesh filename=package://elite_description/meshes/ec63/link3.STL; visual mesh filename=package://elite_description/meshes/ec63/link3.STL
- added link link4, mass 0.53436; collision mesh filename=package://elite_description/meshes/ec63/link4.STL; visual mesh filename=package://elite_description/meshes/ec63/link4.STL
- added link link5, mass 0.53436; collision mesh filename=package://elite_description/meshes/ec63/link5.STL; visual mesh filename=package://elite_description/meshes/ec63/link5.STL
- added link link6, mass 0.16467; collision mesh filename=package://elite_description/meshes/ec63/link6.STL; visual mesh filename=package://elite_description/meshes/ec63/link6.STL
- added link world
Joints:
- added joint flan_joint: type fixed, parent link6, child flan, origin xyz=0 0 0 rpy=0 0 0
- added joint joint1: type revolute, parent base_link, child link1, origin xyz=0 0 0.14 rpy=0 0 0, axis 0 0 1, limit lower=-6.2832 upper=6.2832 effort=90 velocity=3.3161
- added joint joint2: type revolute, parent link1, child link2, origin xyz=0 0 0 rpy=-1.5708 0 0, axis 0 0 1, limit lower=-6.2832 upper=6.2832 effort=90 velocity=3.3161
- added joint joint3: type revolute, parent link2, child link3, origin xyz=0.27 0 0 rpy=0 0 0, axis 0 0 1, limit lower=-2.7925 upper=2.7925 effort=90 velocity=3.3161
- added joint joint4: type revolute, parent link3, child link4, origin xyz=0.256 0 0 rpy=0 0 0, axis 0 0 1, limit lower=-6.2832 upper=6.2832 effort=20 velocity=4.5379
- added joint joint5: type revolute, parent link4, child link5, origin xyz=0 0 0.103 rpy=-1.5708 0 0, axis 0 0 1, limit lower=-6.2832 upper=6.2832 effort=20 velocity=4.5379
- added joint joint6: type revolute, parent link5, child link6, origin xyz=0 0.089 0.098 rpy=-1.5708 0 0, axis 0 0 1, limit lower=-6.2832 upper=6.2832 effort=20 velocity=4.5379
- added joint world_joint: type fixed, parent world, child base_link, origin xyz=0 0 0 rpy=0 0 0
